File: mm_external_uart.kicad_sch (KiCad schematic)
At the start: 0 parts

Commit message: tp02
Parts:
- added J4: Conn_01x04, symbol Connector_Generic:Conn_01x04
- added R19: R, symbol Device:R
Connections:
- new net: J4.3 (Pin_3), R19.2
- new net +BATT: J4.2 (Pin_2)
- new net External_uart Rx: J4.4 (Pin_4)
- new net External_uart Tx: R19.1
- new net GND: J4.1 (Pin_1)
Changed lines of the file:
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@@
 (kicad_sch (version 20230121) (generator eeschema)
   (paper "A4")
+  (wire (pts (xy 149.86 93.98) (xy 152.4 93.98))
+    (stroke (width 0) (type default))
+  )
+  (wire (pts (xy 139.7 93.98) (xy 142.24 93.98))
+    (stroke (width 0) (type default))
+  )
+  (wire (pts (xy 130.81 88.9) (xy 152.4 88.9))
+    (stroke (width 0) (type default))
+  )
+  (wire (pts (xy 127 91.44) (xy 152.4 91.44))
+    (stroke (width 0) (type default))
+  )
+  (wire (pts (xy 139.7 96.52) (xy 152.4 96.52))
+    (stroke (width 0) (type default))
+  )
+  (hierarchical_label "External_uart Tx" (shape output) (at 139.7 93.98 180) (fields_autoplaced)
+    (effects (font (size 1.27 1.27)) (justify right))
+  )
+  (hierarchical_label "External_uart Rx" (shape input) (at 139.7 96.52 180) (fields_autoplaced)
+    (effects (font (size 1.27 1.27)) (justify right))
+  )
+  (symbol (lib_id "Device:R") (at 146.05 93.98 90) (unit 1)
+    (in_bom yes) (on_board yes) (dnp no) (fields_autoplaced)
+    (property "Reference" "R19" (at 146.05 87.63 90)
+      (effects (font (size 1.27 1.27)))
+    )
+    (property "Value" "R" (at 146.05 90.17 90)
+      (effects (font (size 1.27 1.27)))
+    )
+    (property "Footprint" "" (at 146.05 95.758 90)
+      (effects (font (size 1.27 1.27)) hide)
+    )
+    (property "Datasheet" "~" (at 146.05 93.98 0)
+      (effects (font (size 1.27 1.27)) hide)
+    )
+    (pin "1")
+    (pin "2")
+    (instances
+      (project "minimouse"
+        (path "/d8fa4cba-2469-4231-847f-065b6b829f44/d17bb1c7-f68a-465e-9a17-5858ef86fc30"
+          (reference "R19") (unit 1)
+        )
+      )
+    )
+  )
+  (symbol (lib_id "power:+BATT") (at 127 91.44 90) (unit 1)
+    (in_bom yes) (on_board yes) (dnp no) (fields_autoplaced)
+    (property "Reference" "#PWR036" (at 130.81 91.44 0)
+      (effects (font (size 1.27 1.27)) hide)
+    )
+    (property "Value" "+BATT" (at 123.19 91.44 90)
+      (effects (font (size 1.27 1.27)) (justify left))
+    )
+    (property "Footprint" "" (at 127 91.44 0)
+      (effects (font (size 1.27 1.27)) hide)
+    )
+    (property "Datasheet" "" (at 127 91.44 0)
+      (effects (font (size 1.27 1.27)) hide)
+    )
+    (pin "1")
+    (instances
+      (project "minimouse"
+        (path "/d8fa4cba-2469-4231-847f-065b6b829f44/3f9b0845-5778-418c-a7a8-03da2392145e"
+          (reference "#PWR036") (unit 1)
+        )
+        (path "/d8fa4cba-2469-4231-847f-065b6b829f44/d17bb1c7-f68a-465e-9a17-5858ef86fc30"
+          (reference "#PWR017") (unit 1)
+        )
+      )
+    )
+  )
+  (symbol (lib_id "power:GND") (at 130.81 88.9 270) (unit 1)
+    (in_bom yes) (on_board yes) (dnp no) (fields_autoplaced)
+    (property "Reference" "#PWR014" (at 124.46 88.9 0)
+      (effects (font (size 1.27 1.27)) hide)
+    )
+    (property "Value" "GND" (at 127 88.9 90)
+      (effects (font (size 1.27 1.27)) (justify right))
+    )
+    (property "Footprint" "" (at 130.81 88.9 0)
+      (effects (font (size 1.27 1.27)) hide)
+    )
+    (property "Datasheet" "" (at 130.81 88.9 0)
+      (effects (font (size 1.27 1.27)) hide)
+    )
+    (pin "1")
+    (instances
+      (project "minimouse"
+        (path "/d8fa4cba-2469-4231-847f-065b6b829f44/d17bb1c7-f68a-465e-9a17-5858ef86fc30"
+          (reference "#PWR014") (unit 1)
+        )
+      )
+    )
+  )
+  (symbol (lib_id "Connector_Generic:Conn_01x04") (at 157.48 91.44 0) (unit 1)
+    (in_bom yes) (on_board yes) (dnp no)
+    (property "Reference" "J4" (at 162.56 91.44 0)
+      (effects (font (size 1.27 1.27)) (justify left))
+    )
+    (property "Value" "Conn_01x04" (at 160.02 93.98 0)
+      (effects (font (size 1.27 1.27)) (justify left))
+    )
+    (property "Footprint" "" (at 157.48 91.44 0)
+      (effects (font (size 1.27 1.27)) hide)
+    )
+    (property "Datasheet" "~" (at 157.48 91.44 0)
+      (effects (font (size 1.27 1.27)) hide)
+    )
+    (pin "2")
+    (pin "1")
+    (pin "3")
+    (pin "4")
+    (instances
+      (project "minimouse"
+        (path "/d8fa4cba-2469-4231-847f-065b6b829f44/d17bb1c7-f68a-465e-9a17-5858ef86fc30"
+          (reference "J4") (unit 1)
+        )
+      )
+    )
+  )
 )

Commit message: tp3
Parts:
- added C15: 2.2uF, Capacitor_SMD:C_0603_1608Metric, symbol Device:C
- J4: footprint (none) -> Connector_PinHeader_2.54mm:PinHeader_1x04_P2.54mm_Vertical
- R19: value R -> 100; footprint (none) -> Resistor_SMD:R_0603_1608Metric
Connections:
- net +BATT: now also C15.1
- net GND: now also C15.2
- net External_uart Rx renamed EXT_UART_RX
- net External_uart Tx renamed EXT_UART_TX
Other:
- moved on the sheet: R19
Changed lines of the file:
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@@
 (kicad_sch (version 20230121) (generator eeschema)
   (paper "A4")
-  (wire (pts (xy 149.86 93.98) (xy 152.4 93.98))
+  (wire (pts (xy 194.31 82.55) (xy 194.31 91.44))
     (stroke (width 0) (type default))
   )
-  (wire (pts (xy 139.7 93.98) (xy 142.24 93.98))
+  (wire (pts (xy 148.59 93.98) (xy 152.4 93.98))
     (stroke (width 0) (type default))
   )
-  (wire (pts (xy 130.81 88.9) (xy 152.4 88.9))
+  (wire (pts (xy 139.7 93.98) (xy 140.97 93.98))
     (stroke (width 0) (type default))
   )
-  (wire (pts (xy 127 91.44) (xy 152.4 91.44))
+  (wire (pts (xy 149.86 88.9) (xy 152.4 88.9))
+    (stroke (width 0) (type default))
+  )
+  (wire (pts (xy 151.13 91.44) (xy 151.13 80.01))
+    (stroke (width 0) (type default))
+  )
+  (wire (pts (xy 149.86 88.9) (xy 149.86 107.95))
+    (stroke (width 0) (type default))
+  )
+  (wire (pts (xy 194.31 66.04) (xy 194.31 74.93))
+    (stroke (width 0) (type default))
+  )
+  (wire (pts (xy 151.13 91.44) (xy 152.4 91.44))
     (stroke (width 0) (type default))
   )
@@
     (stroke (width 0) (type default))
   )
-  (hierarchical_label "External_uart Tx" (shape output) (at 139.7 93.98 180) (fields_autoplaced)
+  (hierarchical_label "EXT_UART_TX" (shape output) (at 139.7 93.98 180) (fields_autoplaced)
     (effects (font (size 1.27 1.27)) (justify right))
   )
-  (hierarchical_label "External_uart Rx" (shape input) (at 139.7 96.52 180) (fields_autoplaced)
+  (hierarchical_label "EXT_UART_RX" (shape input) (at 139.7 96.52 180) (fields_autoplaced)
     (effects (font (size 1.27 1.27)) (justify right))
   )
-  (symbol (lib_id "Device:R") (at 146.05 93.98 90) (unit 1)
+  (symbol (lib_id "Device:R") (at 144.78 93.98 90) (unit 1)
     (in_bom yes) (on_board yes) (dnp no) (fields_autoplaced)
-    (property "Reference" "R19" (at 146.05 87.63 90)
+    (property "Reference" "R19" (at 144.78 87.63 90)
       (effects (font (size 1.27 1.27)))
     )
-    (property "Value" "R" (at 146.05 90.17 90)
+    (property "Value" "100" (at 144.78 90.17 90)
       (effects (font (size 1.27 1.27)))
     )
-    (property "Footprint" "" (at 146.05 95.758 90)
+    (property "Footprint" "Resistor_SMD:R_0603_1608Metric" (at 144.78 95.758 90)
       (effects (font (size 1.27 1.27)) hide)
     )
-    (property "Datasheet" "~" (at 146.05 93.98 0)
+    (property "Datasheet" "~" (at 144.78 93.98 0)
       (effects (font (size 1.27 1.27)) hide)
     )
@@
     )
   )
-  (symbol (lib_id "power:+BATT") (at 127 91.44 90) (unit 1)
+  (symbol (lib_id "power:+BATT") (at 151.13 80.01 0) (unit 1)
     (in_bom yes) (on_board yes) (dnp no) (fields_autoplaced)
-    (property "Reference" "#PWR036" (at 130.81 91.44 0)
+    (property "Reference" "#PWR017" (at 151.13 83.82 0)
       (effects (font (size 1.27 1.27)) hide)
     )
-    (property "Value" "+BATT" (at 123.19 91.44 90)
-      (effects (font (size 1.27 1.27)) (justify left))
+    (property "Value" "+BATT" (at 151.13 74.93 0)
+      (effects (font (size 1.27 1.27)))
     )
-    (property "Footprint" "" (at 127 91.44 0)
+    (property "Footprint" "" (at 151.13 80.01 0)
       (effects (font (size 1.27 1.27)) hide)
     )
-    (property "Datasheet" "" (at 127 91.44 0)
+    (property "Datasheet" "" (at 151.13 80.01 0)
       (effects (font (size 1.27 1.27)) hide)
     )
@@
     (instances
       (project "minimouse"
-        (path "/d8fa4cba-2469-4231-847f-065b6b829f44/3f9b0845-5778-418c-a7a8-03da2392145e"
-          (reference "#PWR036") (unit 1)
-        )
         (path "/d8fa4cba-2469-4231-847f-065b6b829f44/d17bb1c7-f68a-465e-9a17-5858ef86fc30"
           (reference "#PWR017") (unit 1)
@@
     )
   )
-  (symbol (lib_id "power:GND") (at 130.81 88.9 270) (unit 1)
+  (symbol (lib_id "power:GND") (at 194.31 91.44 0) (unit 1)
     (in_bom yes) (on_board yes) (dnp no) (fields_autoplaced)
-    (property "Reference" "#PWR014" (at 124.46 88.9 0)
+    (property "Reference" "#PWR034" (at 194.31 97.79 0)
       (effects (font (size 1.27 1.27)) hide)
     )
-    (property "Value" "GND" (at 127 88.9 90)
-      (effects (font (size 1.27 1.27)) (justify right))
+    (property "Value" "GND" (at 194.31 96.52 0)
+      (effects (font (size 1.27 1.27)))
     )
-    (property "Footprint" "" (at 130.81 88.9 0)
+    (property "Footprint" "" (at 194.31 91.44 0)
       (effects (font (size 1.27 1.27)) hide)
     )
-    (property "Datasheet" "" (at 130.81 88.9 0)
+    (property "Datasheet" "" (at 194.31 91.44 0)
+      (effects (font (size 1.27 1.27)) hide)
+    )
+    (pin "1")
+    (instances
+      (project "minimouse"
+        (path "/d8fa4cba-2469-4231-847f-065b6b829f44/d17bb1c7-f68a-465e-9a17-5858ef86fc30"
+          (reference "#PWR034") (unit 1)
+        )
+      )
+    )
+  )
+  (symbol (lib_id "Device:C") (at 194.31 78.74 0) (unit 1)
+    (in_bom yes) (on_board yes) (dnp no) (fields_autoplaced)
+    (property "Reference" "C15" (at 198.12 77.47 0)
+      (effects (font (size 1.27 1.27)) (justify left))
+    )
+    (property "Value" "2.2uF" (at 198.12 80.01 0)
+      (effects (font (size 1.27 1.27)) (justify left))
+    )
+    (property "Footprint" "Capacitor_SMD:C_0603_1608Metric" (at 195.2752 82.55 0)
+      (effects (font (size 1.27 1.27)) hide)
+    )
+    (property "Datasheet" "~" (at 194.31 78.74 0)
+      (effects (font (size 1.27 1.27)) hide)
+    )
+    (pin "2")
+    (pin "1")
+    (instances
+      (project "minimouse"
+        (path "/d8fa4cba-2469-4231-847f-065b6b829f44/d17bb1c7-f68a-465e-9a17-5858ef86fc30"
+          (reference "C15") (unit 1)
+        )
+      )
+    )
+  )
+  (symbol (lib_id "power:+BATT") (at 194.31 66.04 0) (unit 1)
+    (in_bom yes) (on_board yes) (dnp no) (fields_autoplaced)
+    (property "Reference" "#PWR033" (at 194.31 69.85 0)
+      (effects (font (size 1.27 1.27)) hide)
+    )
+    (property "Value" "+BATT" (at 194.31 60.96 0)
+      (effects (font (size 1.27 1.27)))
+    )
+    (property "Footprint" "" (at 194.31 66.04 0)
+      (effects (font (size 1.27 1.27)) hide)
+    )
+    (property "Datasheet" "" (at 194.31 66.04 0)
+      (effects (font (size 1.27 1.27)) hide)
+    )
+    (pin "1")
+    (instances
+      (project "minimouse"
+        (path "/d8fa4cba-2469-4231-847f-065b6b829f44/d17bb1c7-f68a-465e-9a17-5858ef86fc30"
+          (reference "#PWR033") (unit 1)
+        )
+      )
+    )
+  )
+  (symbol (lib_id "power:GND") (at 149.86 107.95 0) (unit 1)
+    (in_bom yes) (on_board yes) (dnp no) (fields_autoplaced)
+    (property "Reference" "#PWR014" (at 149.86 114.3 0)
+      (effects (font (size 1.27 1.27)) hide)
+    )
+    (property "Value" "GND" (at 149.86 113.03 0)
+      (effects (font (size 1.27 1.27)))
+    )
+    (property "Footprint" "" (at 149.86 107.95 0)
+      (effects (font (size 1.27 1.27)) hide)
+    )
+    (property "Datasheet" "" (at 149.86 107.95 0)
       (effects (font (size 1.27 1.27)) hide)
     )
@@
       (effects (font (size 1.27 1.27)) (justify left))
     )
-    (property "Footprint" "" (at 157.48 91.44 0)
+    (property "Footprint" "Connector_PinHeader_2.54mm:PinHeader_1x04_P2.54mm_Vertical" (at 157.48 91.44 0)
       (effects (font (size 1.27 1.27)) hide)
     )
