File: mm_motor.kicad_sch (KiCad schematic)
At the start: 1 part, among them M1 N20_encoder

Commit message: tp02
Parts:
- added J2: Conn_01x06, symbol Connector_Generic:Conn_01x06
Connections:
- net C1: now also J2.3 (Pin_3)
- net C2: now also J2.4 (Pin_4)
- net MA: now also J2.1 (Pin_1)
- net MB: now also J2.6 (Pin_6)
- new net +BATT: J2.5 (Pin_5)
- new net GND: J2.2 (Pin_2)
Changed lines of the file:
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@@
 (kicad_sch (version 20230121) (generator eeschema)
   (paper "A4")
+  (wire (pts (xy 118.11 93.98) (xy 123.19 93.98))
+    (stroke (width 0) (type default))
+  )
+  (wire (pts (xy 113.03 96.52) (xy 123.19 96.52))
+    (stroke (width 0) (type default))
+  )
+  (wire (pts (xy 118.11 99.06) (xy 123.19 99.06))
+    (stroke (width 0) (type default))
+  )
+  (wire (pts (xy 118.11 91.44) (xy 123.19 91.44))
+    (stroke (width 0) (type default))
+  )
+  (wire (pts (xy 110.49 88.9) (xy 123.19 88.9))
+    (stroke (width 0) (type default))
+  )
+  (wire (pts (xy 118.11 86.36) (xy 123.19 86.36))
+    (stroke (width 0) (type default))
+  )
   (hierarchical_label "C1" (shape output) (at 118.11 91.44 180) (fields_autoplaced)
     (effects (font (size 1.27 1.27)) (justify right))
@@
   (hierarchical_label "MA" (shape passive) (at 118.11 86.36 180) (fields_autoplaced)
     (effects (font (size 1.27 1.27)) (justify right))
+  )
+  (symbol (lib_id "power:+BATT") (at 113.03 96.52 90) (unit 1)
+    (in_bom yes) (on_board yes) (dnp no) (fields_autoplaced)
+    (property "Reference" "#PWR036" (at 116.84 96.52 0)
+      (effects (font (size 1.27 1.27)) hide)
+    )
+    (property "Value" "+BATT" (at 109.22 96.52 90)
+      (effects (font (size 1.27 1.27)) (justify left))
+    )
+    (property "Footprint" "" (at 113.03 96.52 0)
+      (effects (font (size 1.27 1.27)) hide)
+    )
+    (property "Datasheet" "" (at 113.03 96.52 0)
+      (effects (font (size 1.27 1.27)) hide)
+    )
+    (pin "1")
+    (instances
+      (project "minimouse"
+        (path "/d8fa4cba-2469-4231-847f-065b6b829f44/3f9b0845-5778-418c-a7a8-03da2392145e"
+          (reference "#PWR036") (unit 1)
+        )
+        (path "/d8fa4cba-2469-4231-847f-065b6b829f44/7f113667-692a-4f4d-b16f-621d32f3f136"
+          (reference "#PWR015") (unit 1)
+        )
+        (path "/d8fa4cba-2469-4231-847f-065b6b829f44/3975acd0-18ad-47bc-9ce1-d8c4d864aafe"
+          (reference "#PWR016") (unit 1)
+        )
+      )
+    )
+  )
+  (symbol (lib_id "power:GND") (at 110.49 88.9 270) (unit 1)
+    (in_bom yes) (on_board yes) (dnp no) (fields_autoplaced)
+    (property "Reference" "#PWR08" (at 104.14 88.9 0)
+      (effects (font (size 1.27 1.27)) hide)
+    )
+    (property "Value" "GND" (at 106.68 88.9 90)
+      (effects (font (size 1.27 1.27)) (justify right))
+    )
+    (property "Footprint" "" (at 110.49 88.9 0)
+      (effects (font (size 1.27 1.27)) hide)
+    )
+    (property "Datasheet" "" (at 110.49 88.9 0)
+      (effects (font (size 1.27 1.27)) hide)
+    )
+    (pin "1")
+    (instances
+      (project "minimouse"
+        (path "/d8fa4cba-2469-4231-847f-065b6b829f44/7f113667-692a-4f4d-b16f-621d32f3f136"
+          (reference "#PWR08") (unit 1)
+        )
+        (path "/d8fa4cba-2469-4231-847f-065b6b829f44/3975acd0-18ad-47bc-9ce1-d8c4d864aafe"
+          (reference "#PWR09") (unit 1)
+        )
+      )
+    )
   )
   (symbol (lib_id "minimouse:N20_w_encoder") (at 115.57 57.15 0) (unit 1)
@@
         )
       )
+    )
+  )
+  (symbol (lib_id "Connector_Generic:Conn_01x06") (at 128.27 91.44 0) (unit 1)
+    (in_bom yes) (on_board yes) (dnp no) (fields_autoplaced)
+    (property "Reference" "J2" (at 130.81 91.44 0)
+      (effects (font (size 1.27 1.27)) (justify left))
+    )
+    (property "Value" "Conn_01x06" (at 130.81 93.98 0)
+      (effects (font (size 1.27 1.27)) (justify left))
+    )
+    (property "Footprint" "" (at 128.27 91.44 0)
+      (effects (font (size 1.27 1.27)) hide)
+    )
+    (property "Datasheet" "~" (at 128.27 91.44 0)
+      (effects (font (size 1.27 1.27)) hide)
+    )
+    (pin "2")
+    (pin "4")
+    (pin "3")
+    (pin "6")
+    (pin "1")
+    (pin "5")
+    (instances
+      (project "minimouse"
+        (path "/d8fa4cba-2469-4231-847f-065b6b829f44/7f113667-692a-4f4d-b16f-621d32f3f136"
+          (reference "J2") (unit 1)
+        )
+        (path "/d8fa4cba-2469-4231-847f-065b6b829f44/3975acd0-18ad-47bc-9ce1-d8c4d864aafe"
+          (reference "J3") (unit 1)
+        )
+      )

Commit message: tp3
Parts:
- added C7: 2.2uF, Capacitor_SMD:C_0603_1608Metric, symbol Device:C
- added R18, R22: 100, Resistor_SMD:R_0603_1608Metric, symbol Device:R
- J2: footprint (none) -> Connector_PinHeader_2.54mm:PinHeader_1x06_P2.54mm_Vertical
Connections:
- net +BATT: now also C7.1
- net C1: now also R18.1; no longer J2.3 (Pin_3)
- net C2: now also R22.1; no longer J2.4 (Pin_4)
- net GND: now also C7.2
- new net: J2.4 (Pin_4), R22.2
- new net: J2.3 (Pin_3), R18.2
Other:
- moved on the sheet: M1
