File: mm_motor_control.kicad_sch (KiCad schematic)
At the start: 0 parts

Commit message: tp02
Parts:
- added C10: 22 nF, symbol Device:C
- added C11: 10nF, symbol Device:C
- added C12: 1 nF, symbol Device:C
- added C7: C, symbol Device:C
- added C8: 2.2 µF, symbol Device:C
- added R10, R16, R17: R, symbol Device:R
- added R11: 1 kΩ, symbol Device:R
- added R12: 47 kΩ, symbol Device:R
- added R13, R14: 330mΩ, symbol Device:R
- added R15, R18: 18 kΩ, symbol Device:R
- added U3: STSPIN240, Package_DFN_QFN:VQFN-16-1EP_3x3mm_P0.5mm_EP1.8x1.8mm, symbol Driver_Motor:STSPIN240
Connections:
- net EN: now also R15.1
- net FAULT: now also C11.1, R15.2, U3.13 (EN/FLT)
- net OUT_A1: now also U3.3 (OUTA1)
- net OUT_A2: now also U3.5 (OUTA2)
- net OUT_B1: now also U3.10 (OUTB1)
- net OUT_B2: now also U3.8 (OUTB2)
- net PHASE_A: now also U3.1 (PHA)
- net PHASE_B: now also U3.15 (PHB)
- net PWM_A: now also U3.2 (PWMA)
- net PWM_B: now also U3.16 (PWMB)
- net STBY/RESET: now also C12.1, R18.2, U3.14 (STBY/RESET)
- new net: C10.1, R11.2, R12.2
- new net: R14.1, U3.4 (SENSEA)
- new net: R13.1, U3.9 (SENSEB)
- new net: C7.1, R10.1, U3.11 (REF)
- new net: R10.2, R16.2, R17.1
- new net: R11.1, R12.1, U3.12 (TOFF)
- new net GND: C10.2, C11.2, C12.2, C7.2, C8.1, C8.2, R13.2, R14.2, R16.1, R17.2, U3.6 (VS), U3.7 (GND)
- new net VDD: R18.1

Commit message: tp3
Parts:
- removed C12: 1 nF, symbol Device:C
- removed C7: C, symbol Device:C
- removed C8: 2.2 µF, symbol Device:C
- removed R10: R, symbol Device:R
- removed R18: 18 kΩ, symbol Device:R
- added C16: 2.2uF, Capacitor_SMD:C_0603_1608Metric, symbol Device:C
- C10: footprint (none) -> Capacitor_SMD:C_0603_1608Metric
- C11: value 10nF -> 1nF; footprint (none) -> Capacitor_SMD:C_0603_1608Metric
- R11, R12: footprint (none) -> Resistor_SMD:R_0603_1608Metric
- R13, R14: footprint (none) -> Resistor_SMD:R_2512_6332Metric
- R15: value 18 kΩ -> 10kΩ; footprint (none) -> Resistor_SMD:R_0603_1608Metric
- R16, R17: value R -> 10k; footprint (none) -> Resistor_SMD:R_0603_1608Metric
Connections:
- net GND: now also R12.2, U3.17 (EPAD), C16.2; no longer R16.1, U3.6 (VS)
- net at C10.1, R11.2: no longer R12.2
- net at U3.11 (REF): now also R16.2, R17.1
- new net +BATT: C16.1, R16.1, U3.6 (VS)
Other:
- moved on the sheet: C11, R14, R15, R16, R17
