File: mm_power.kicad_sch (KiCad schematic)
At the start: 1 part, among them J5 Conn_01x02

Commit message: tp02
Parts:
- added U2: LP5907MFX-3.3, Package_TO_SOT_SMD:SOT-23-5, symbol Regulator_Linear:LP5907MFX-3.3
Connections:
- net GND: now also U2.2 (GND)
Changed lines of the file:
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@@
   (junction (at 86.36 95.25) (diameter 0) (color 0 0 0 0)
   )
+  (junction (at 86.36 97.79) (diameter 0) (color 0 0 0 0)
+  )
   (wire (pts (xy 86.36 90.17) (xy 86.36 95.25))
+    (stroke (width 0) (type default))
+  )
+  (wire (pts (xy 36.83 97.79) (xy 86.36 97.79))
     (stroke (width 0) (type default))
   )
@@
     (stroke (width 0) (type default))
   )
-  (wire (pts (xy 86.36 95.25) (xy 86.36 100.33))
+  (wire (pts (xy 86.36 95.25) (xy 86.36 97.79))
     (stroke (width 0) (type default))
   )
@@
     (stroke (width 0) (type default))
   )
+  (wire (pts (xy 86.36 97.79) (xy 86.36 100.33))
+    (stroke (width 0) (type default))
+  )
   (wire (pts (xy 86.36 82.55) (xy 86.36 87.63))
+    (stroke (width 0) (type default))
+  )
+  (wire (pts (xy 36.83 85.09) (xy 36.83 97.79))
     (stroke (width 0) (type default))
   )
@@
         )
       )
+    )
+  )
+  (symbol (lib_id "Regulator_Linear:LP5907MFX-3.3") (at 36.83 77.47 0) (unit 1)
+    (in_bom yes) (on_board yes) (dnp no) (fields_autoplaced)
+    (property "Reference" "U2" (at 36.83 67.31 0)
+      (effects (font (size 1.27 1.27)))
+    )
+    (property "Value" "LP5907MFX-3.3" (at 36.83 69.85 0)
+      (effects (font (size 1.27 1.27)))
+    )
+    (property "Footprint" "Package_TO_SOT_SMD:SOT-23-5" (at 36.83 68.58 0)
+      (effects (font (size 1.27 1.27)) hide)
+    )
+    (property "Datasheet" "http://www.ti.com/lit/ds/symlink/lp5907.pdf" (at 36.83 64.77 0)
+      (effects (font (size 1.27 1.27)) hide)
+    )
+    (pin "3")
+    (pin "5")
+    (pin "4")
+    (pin "2")
+    (pin "1")
+    (instances
+      (project "minimouse"
+        (path "/d8fa4cba-2469-4231-847f-065b6b829f44/3f9b0845-5778-418c-a7a8-03da2392145e"
+          (reference "U2") (unit 1)
+        )
+      )

Commit message: tp3
Parts:
- added C13, C14: 2.2uF, Capacitor_SMD:C_0603_1608Metric, symbol Device:C
- added D1: LED, LED_SMD:LED_0603_1608Metric, symbol Device:LED
- added R21: 330, Resistor_SMD:R_0603_1608Metric, symbol Device:R
Connections:
- net +BATT: now also U2.1 (IN), U2.3 (EN), C14.1
- net GND: now also C13.2, C14.2, D1.1 (K)
- net +3.3V: now reaches U2.5 (OUT)
- net +3.3V: now also C13.1, R21.1
- new net: D1.2 (A), R21.2
Other:
- moved on the sheet: U2
