File: minimouse.kicad_pcb (KiCad board)
At the start: 2 copper layers, 90 x 85 mm, 22 parts, among them J1 Conn_ARM_JTAG_SWD_10, J5 Conn_01x02, M1 N20_encoder, M2 N20_encoder, U1 STM32F030C8Tx, U4 HC-SR04

Commit message: tp3
Parts:
- added C10: 22 nF, Capacitor_SMD:C_0603_1608Metric, F.Cu at (132.2, 91.6)
- added C11: 1nF, Capacitor_SMD:C_0603_1608Metric, F.Cu at (144.9, 103.3)
- added C12: 2.2uF, Capacitor_SMD:C_0603_1608Metric, F.Cu at (170.3, 87.3)
- added C13: 2.2uF, Capacitor_SMD:C_0603_1608Metric, F.Cu at (178.0, 87.3)
- added C14: 2.2uF, Capacitor_SMD:C_0603_1608Metric, F.Cu at (180.5, 87.3)
- added C15: 2.2uF, Capacitor_SMD:C_0603_1608Metric, F.Cu at (117.0, 87.3)
- added C16: 2.2uF, Capacitor_SMD:C_0603_1608Metric, F.Cu at (177.9, 71.3)
- added C7: 2.2uF, Capacitor_SMD:C_0603_1608Metric, F.Cu at (162.7, 98.3)
- added C9: 2.2 uF, Capacitor_SMD:C_0603_1608Metric, F.Cu at (158.4, 79.7)
- added D1: LED, LED_SMD:LED_0603_1608Metric, F.Cu at (187.3, 94.9)
- added J2: Conn_01x06, Connector_PinHeader_2.54mm:PinHeader_1x06_P2.54mm_Vertical, F.Cu at (162.7, 102.5)
- added J3: Conn_01x06, Connector_PinHeader_2.54mm:PinHeader_1x06_P2.54mm_Vertical, F.Cu at (124.6, 102.5)
- added J4: Conn_01x04, Connector_PinHeader_2.54mm:PinHeader_1x04_P2.54mm_Vertical, F.Cu at (122.1, 81.0)
- added R10: 100, Resistor_SMD:R_0603_1608Metric, F.Cu at (167.8, 98.3)
- added R11: 1 kΩ, Resistor_SMD:R_0603_1608Metric, F.Cu at (132.2, 96.6)
- added R12: 47 kΩ, Resistor_SMD:R_0603_1608Metric, F.Cu at (134.8, 96.6)
- added R13: 330mΩ, Resistor_SMD:R_2512_6332Metric, F.Cu at (157.6, 112.7)
- added R14: 330mΩ, Resistor_SMD:R_2512_6332Metric, F.Cu at (142.0, 112.7)
- added R15: 10kΩ, Resistor_SMD:R_0603_1608Metric, F.Cu at (142.4, 103.4)
- added R16: 10k, Resistor_SMD:R_0603_1608Metric, F.Cu at (137.3, 96.6)
- added R17: 10k, Resistor_SMD:R_0603_1608Metric, F.Cu at (139.8, 96.6)
- added R18: 100, Resistor_SMD:R_0603_1608Metric, F.Cu at (124.6, 98.3)
- added R19: 100, Resistor_SMD:R_0603_1608Metric, F.Cu at (129.7, 87.3)
- added R20: 100, Resistor_SMD:R_0603_1608Metric, F.Cu at (158.4, 82.2)
- added R21: 330, Resistor_SMD:R_0603_1608Metric, F.Cu at (183.0, 87.3)
- added R22: 100, Resistor_SMD:R_0603_1608Metric, F.Cu at (170.3, 98.3)
- added R23: 100, Resistor_SMD:R_0603_1608Metric, F.Cu at (127.1, 98.3)
- added U2: LP5907MFX-3.3, Package_TO_SOT_SMD:SOT-23-5, F.Cu at (179.3, 93.3)
- added U3: STSPIN240, Package_DFN_QFN:VQFN-16-1EP_3x3mm_P0.5mm_EP1.8x1.8mm, F.Cu at (148.5, 106.9)
- moved R7 20.5 mm to (139.8, 83.0)
- moved C6 13.9 mm to (129.7, 81.4)
- moved C2 13.0 mm to (132.2, 81.4)
- moved R3 11.6 mm to (153.6, 104.3)
- moved R4 11.6 mm to (155.1, 104.3)
- moved R5 11.6 mm to (156.6, 104.3)
- moved C5 7.04 mm to (119.5, 94.9)
- moved BOOT0 6.79 mm to (160.2, 72.1)
- moved R1 2.14 mm to (149.4, 78.9)
- moved R8 2.14 mm to (151.3, 78.9)
- moved R9 2.14 mm to (147.1, 79.0)
- moved R6 2.01 mm to (152.5, 99.2)
- moved R2 1.19 mm to (142.4, 96.6)
- moved J1 0.30 mm to (163.9, 83.5)
Connections:
- R8 pad 1: /mcu/UART1_TX -> /external_uart/EXT_UART_RX
- U1 pad 43: /mcu/UART1_RX -> /external_uart/EXT_UART_TX
- U4 pad 4: +3V3 -> +3.3V
Routing:
- net Net-(J4-Pin_3): track 0.00 -> 8.97 mm

Commit message: tp33
Parts:
- moved C16 1.55 mm to (177.9, 72.8)
- moved R9 0.39 mm to (147.5, 78.9)
Routing:
- net Net-(J4-Pin_3): track 8.97 -> 0.00 mm
Changed lines of the file:
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@@
   )
   (footprint "Resistor_SMD:R_0603_1608Metric" (layer "F.Cu")
-    (at 147.0875 78.955 -90)
+    (at 147.46 78.855 -90)
     (descr "Resistor SMD 0603 (1608 Metric), square (rectangular) end terminal, IPC_7351 nominal, (Body size source: IPC-SM-782 page 72, https://www.pcb-3d.com/wordpress/wp-content/uploads/ipc-sm-782a_amendment_1_and_2.pdf), generated with kicad-footprint-generator")
     (tags "resistor")
@@
     (property "ki_keywords" "R res resistor")
     (attr smd)
-    (fp_text reference "R9" (at 0 -1.43 90) (layer "F.SilkS")
+    (fp_text reference "R9" (at 0.237258 0.5225 90) (layer "F.SilkS")
         (effects (font (size 1 1) (thickness 0.15)))
     )
@@
   )
   (footprint "Capacitor_SMD:C_0603_1608Metric" (layer "F.Cu")
-    (at 177.94 71.285 90)
+    (at 177.94 72.835 90)
     (descr "Capacitor SMD 0603 (1608 Metric), square (rectangular) end terminal, IPC_7351 nominal, (Body size source: IPC-SM-782 page 76, https://www.pcb-3d.com/wordpress/wp-content/uploads/ipc-sm-782a_amendment_1_and_2.pdf), generated with kicad-footprint-generator")
     (tags "capacitor")
@@
   (gr_line (start 118.5 140) (end 118.5 100)
     (stroke (width 0.2) (type solid)) (layer "Edge.Cuts"))
-  (segment (start 129.245 86.04) (end 130.505 87.3) (width 0.2) (layer "F.Cu") (net 64))
-  (segment (start 122.06 86.04) (end 129.245 86.04) (width 0.2) (layer "F.Cu") (net 64))
   (group "" (id 31bb09ae-506e-485d-9a47-edcfb72f895d)
     (members
